File: hardware/Modbus-Adapter.kicad_pcb (KiCad board)
At the start: 2 copper layers, 27.9 x 41.7 mm, 23 parts, among them J2 USB_C_Receptacle_USB2.0_16P, J3 Conn_01x04_Pin, J4 Conn_01x04_Pin, SW1 SW_Push, SW2 SW_Push, U1 ESP32-C6-MINI-1, U2 MAX3485, U4 AP2112K-3.3

Commit message: Revision B of the PCB
Routing:
- net +5V: vias 2 -> 1
Changed lines of the file:
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@@
 	(title_block
 		(title "Modbus ESP32 Adapter")
-		(date "2026-08-02")
-		(rev "A")
+		(date "2026-08-24")
+		(rev "B")
 		(comment 4 "AISLER Project ID: ZEWTBDOS")
 	)
@@
 		(size 0.6)
 		(drill 0.3)
-		(layers "F.Cu" "B.Cu")
-		(net "+5V")
-	)
-	(via
-		(at 89.134 68.58)
-		(size 0.6)
-		(drill 0.3)
